Commit message: commit spaghetti

File: walker_sim/robots/walker_fake.urdf (robot description, URDF)
Before this commit: robot bipedalWalker, 1 links, 0 joints
Links:
- added link boom, mass 0.18809; collision mesh filename=package://install/walker_sim/share/walker_sim/meshes/boom_h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
- added link footL, mass 0.0098175; collision mesh filename=package://install/walker_sim/share/walker_sim/meshes/contac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; visual mesh filename=package://install/walker_sim/share/walker_sim/meshes/contac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
- added link footR, mass 0.0098175; collision mesh filename=package://install/walker_sim/share/walker_sim/meshes/contac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; visual mesh filename=package://install/walker_sim/share/walker_sim/meshes/contac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
- added link inner_ring, mass 0.41592; collision mesh filename=package://install/walker_sim/share/walker_sim/meshes/inner_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
- added link outer_ring, mass 0.49244; collision mesh filename=package://install/walker_sim/share/walker_sim/meshes/outter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
- added link shankL, mass 0.069508; collision mesh filename=package://install/walker_sim/share/walker_sim/meshes/shank.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; visual mesh filename=package://install/walker_sim/share/walker_sim/meshes/shank.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
- added link shankR, mass 0.069508; collision mesh filename=package://install/walker_sim/share/walker_sim/meshes/shank.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; visual mesh filename=package://install/walker_sim/share/walker_sim/meshes/shank.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
- added link thighL, mass 0.045155; collision mesh filename=package://install/walker_sim/share/walker_sim/meshes/thigh.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; visual mesh filename=package://install/walker_sim/share/walker_sim/meshes/thigh.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
- added link thighR, mass 0.045155; collision mesh filename=package://install/walker_sim/share/walker_sim/meshes/thigh.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; visual mesh filename=package://install/walker_sim/share/walker_sim/meshes/thigh.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
- added link world
- link waist: geometry collision mesh filename=package://install/walker_sim/share/walker_sim/meshes/waist_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; visual mesh filename=package://install/walker_sim/share/walker_sim/meshes/waist_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
Joints:
- added joint boom_waist: type prismatic, parent boom, child waist, origin xyz=0.725 0.0 0.0 rpy=0.0 0.0 0.0, axis 0.0 0.0 1.0, limit lower=-0.5 upper=0.5 effort=30 velocity=7.0
- added joint grounding: type fixed, parent world, child outer_ring, origin xyz=0.0 0.0 0.0 rpy=0.0 0.0 0.0
- added joint inner_ring_boom: type fixed, parent inner_ring, child boom, origin xyz=0 0 0.080 rpy=0.0 0.0 0.0, axis 0 -1 0
- added joint outer_ring_inner_ring: type prismatic, parent outer_ring, child inner_ring, origin xyz=0.0 0.0 0.330 rpy=0.0 0.0 0.0, axis 0 -1 0, limit lower=0.0 upper=10.0 effort=30 velocity=7.0
- added joint shankL_footL: type fixed, parent shankL, child footL, origin xyz=0.0 0.0 -0.175 rpy=0.0 0.0 0.0
- added joint shankR_footR: type fixed, parent shankR, child footR, origin xyz=0.0 0.0 -0.175 rpy=0.0 0.0 0.0
- added joint thighL_shankL: type revolute, parent thighL, child shankL, origin xyz=0.0 0.0 -0.190 rpy=0.0 0.0 0.0, axis 1.0 0.0 0.0, limit lower=-0.00118981 upper=1.4 effort=30 velocity=7.0
- added joint thighR_shankR: type revolute, parent thighR, child shankR, origin xyz=0.0 0.0 -0.190 rpy=0.0 0.0 0.0, axis 1.0 0.0 0.0, limit lower=-0.00118981 upper=1.4 effort=30.0 velocity=7.0
- added joint waist_thighL: type revolute, parent waist, child thighL, origin xyz=0.0775 0.0 0.0 rpy=0.0 0.0 0.0, axis 1.0 0.0 0.0, limit lower=-0.8 upper=0.8 effort=30 velocity=7.0
- added joint waist_thighR: type revolute, parent waist, child thighR, origin xyz=-0.0775 0.0 0.0 rpy=0.0 0.0 0.0, axis 1.0 0.0 0.0, limit lower=-0.8 upper=0.8 effort=30 velocity=7.0
