Commit message: mesh file change

File: walker_sim/robots/simple_walker.urdf (robot description, URDF)
Before this commit: robot bipedal_walker, 11 links, 10 joints
Links:
- link boom: geometry collision mesh filename=file://($find walker_sim)/meshes/boom_horizontal.STL
- link footL: geometry collision mesh filename=file://($find walker_sim)/meshes/contact_sensor.STL; visual mesh filename=file://($find walker_sim)/meshes/contact_sensor.STL
- link footR: geometry collision mesh filename=file://($find walker_sim)/meshes/contact_sensor.STL; visual mesh filename=file://($find walker_sim)/meshes/contact_sensor.STL
- link inner_ring: geometry collision mesh filename=file://($find walker_sim)/meshes/inner_ring.STL
- link outer_ring: geometry collision mesh filename=file://($find walker_sim)/meshes/outter_ring.STL
- link shankL: geometry collision mesh filename=file://($find walker_sim)/meshes/shank.STL; visual mesh filename=file://($find walker_sim)/meshes/shank.STL
- link shankR: geometry collision mesh filename=file://($find walker_sim)/meshes/shank.STL; visual mesh filename=file://($find walker_sim)/meshes/shank.STL
- link thighL: geometry collision mesh filename=file://($find walker_sim)/meshes/31mar/thigh.STL; visual mesh filename=file://($find walker_sim)/meshes/thigh.STL
- link thighR: geometry collision mesh filename=file://($find walker_sim)/meshes/thigh.STL; visual mesh filename=file://($find walker_sim)/meshes/thigh.STL
- link waist: geometry collision mesh filename=file://($find walker_sim)/meshes/waist_L.STL; visual mesh filename=file://($find walker_sim)/meshes/waist_L.STL
