Commit message: got robot working in simple rviz. can this work normal yet?

File: walker_sim/robots/barebones.urdf (robot description, URDF)
Before this commit: robot bipedal_walker, 11 links, 10 joints
Links:
- link boom: geometry collision mesh filename=package://walker_sim/meshes/boom_horizontal.STL
- link footL: geometry collision mesh filename=package://walker_sim/meshes/contact_sensor.STL; visual mesh filename=package://walker_sim/meshes/contact_sensor.STL
- link footR: geometry collision mesh filename=package://walker_sim/meshes/contact_sensor.STL; visual mesh filename=package://walker_sim/meshes/contact_sensor.STL
- link inner_ring: geometry collision mesh filename=package://walker_sim/meshes/inner_ring.STL
- link outer_ring: geometry collision mesh filename=package://walker_sim/meshes/outter_ring.STL
- link shankL: geometry collision mesh filename=package://walker_sim/meshes/shank.STL; visual mesh filename=package://walker_sim/meshes/shank.STL
- link shankR: geometry collision mesh filename=package://walker_sim/meshes/shank.STL; visual mesh filename=package://walker_sim/meshes/shank.STL
- link thighL: geometry collision mesh filename=package://walker_sim/meshes/thigh.STL; visual mesh filename=package://walker_sim/meshes/thigh.STL
- link thighR: geometry collision mesh filename=package://walker_sim/meshes/thigh.STL; visual mesh filename=package://walker_sim/meshes/thigh.STL
- link waist: geometry collision mesh filename=package://walker_sim/meshes/waist_L.STL; visual mesh filename=package://walker_sim/meshes/waist_L.STL
Joints:
- joint boom_waist: axis 0.0 0.0 1.0 -> 0 0 1; origin xyz=0.725 0.0 0.0 rpy=0.0 0.0 0.0 -> xyz=0.725 0 0 rpy=0 0 0
- joint grounding: origin xyz=0.0 0.0 0.0 rpy=0.0 0.0 0.0 -> xyz=0 0 0 rpy=0 0 0
- joint inner_ring_boom: origin xyz=0 0 0.080 rpy=0.0 0.0 0.0 -> xyz=0 0 0.080 rpy=0 0 0
- joint outer_ring_inner_ring: origin xyz=0.0 0.0 0.330 rpy=0.0 0.0 0.0 -> xyz=0 0 0.330 rpy=0 0 0
- joint shankL_footL: origin xyz=0.0 0.0 -0.175 rpy=0.0 0.0 0.0 -> xyz=0 0 -0.175 rpy=0 0 0
- joint shankR_footR: origin xyz=0.0 0.0 -0.175 rpy=0.0 0.0 0.0 -> xyz=0 0 -0.175 rpy=0 0 0
- joint thighL_shankL: axis 1.0 0.0 0.0 -> 1 0 0; origin xyz=0.0 0.0 -0.190 rpy=0.0 0.0 0.0 -> xyz=0 0 -0.190 rpy=0 0 0
- joint thighR_shankR: axis 1.0 0.0 0.0 -> 1 0 0; limit lower=-0.00118981 upper=1.4 effort=30.0 velocity=7.0 -> lower=-0.00118981 upper=1.4 effort=30 velocity=7.0; origin xyz=0.0 0.0 -0.190 rpy=0.0 0.0 0.0 -> xyz=0 0 -0.190 rpy=0 0 0
- joint waist_thighL: axis 1.0 0.0 0.0 -> 1 0 0; origin xyz=0.0775 0.0 0.0 rpy=0.0 0.0 0.0 -> xyz=0.0775 0 0 rpy=0 0 0
- joint waist_thighR: axis 1.0 0.0 0.0 -> 1 0 0; origin xyz=-0.0775 0.0 0.0 rpy=0.0 0.0 0.0 -> xyz=-0.0775 0 0 rpy=0 0 0

File: walker_sim/robots/simple_walker.urdf (robot description, URDF)
Before this commit: robot bipedal_walker, 11 links, 10 joints
Links:
- link boom: geometry collision mesh filename=package://walker_sim/meshes/boom_horizontal.STL
- link footL: geometry collision mesh filename=package://walker_sim/meshes/contact_sensor.STL; visual mesh filename=package://walker_sim/meshes/contact_sensor.STL
- link footR: geometry collision mesh filename=package://walker_sim/meshes/contact_sensor.STL; visual mesh filename=package://walker_sim/meshes/contact_sensor.STL
- link inner_ring: geometry collision mesh filename=package://walker_sim/meshes/inner_ring.STL
- link outer_ring: geometry collision mesh filename=package://walker_sim/meshes/outter_ring.STL
- link shankL: geometry collision mesh filename=package://walker_sim/meshes/shank.STL; visual mesh filename=package://walker_sim/meshes/shank.STL
- link shankR: geometry collision mesh filename=package://walker_sim/meshes/shank.STL; visual mesh filename=package://walker_sim/meshes/shank.STL
- link thighL: geometry collision mesh filename=package://walker_sim/meshes/thigh.STL; visual mesh filename=package://walker_sim/meshes/thigh.STL
- link thighR: geometry collision mesh filename=package://walker_sim/meshes/thigh.STL; visual mesh filename=package://walker_sim/meshes/thigh.STL
- link waist: geometry collision mesh filename=package://walker_sim/meshes/waist_L.STL; visual mesh filename=package://walker_sim/meshes/waist_L.STL

Commit message: cpp reset control client

File: walker_sim/robots/barebones.urdf (robot description, URDF)
Before this commit: robot bipedalwalkingrobot, 11 links, 10 joints
Joints:
- removed joint boom_waist

Commit message: attempt raw control

File: walker_sim/robots/barebones.urdf (robot description, URDF)
Before this commit: robot bipedal_walker, 11 links, 9 joints
Links:
- removed link world

File: walker_sim/robots/simple_walker.urdf (robot description, URDF)
Before this commit: robot bipedal_walker, 11 links, 10 joints
Links:
- removed link world

Commit message: barebones rviz working

File: walker_sim/robots/barebones.urdf (robot description, URDF)
Before this commit: robot bipedal_walker, 10 links, 9 joints
Links:
- added link world
Joints:
- added joint boom_waist: type prismatic, parent boom, child waist, origin xyz=0.725 0 0 rpy=0 0 0, axis 0 0 1, limit lower=-0.5 upper=0.5 effort=30 velocity=7.0

File: walker_sim/robots/simple_walker.urdf (robot description, URDF)
Before this commit: robot bipedal_walker, 10 links, 10 joints
Links:
- added link world
